Commit message: added yanu description

File: urdf/yanu_3.urdf.xacro (robot description, xacro)
@@ -1,5 +1,5 @@
 <?xml version="1.0"?>
 <robot xmlns:xacro="http://www.ros.org/wiki/xacro" name="yanu">
-  <!-- panda -->
+  <!-- panda and its hand-->
   <xacro:include filename="$(find franka_description)/robots/panda/panda.urdf.xacro"/>
   <xacro:include filename="$(find franka_description)/robots/common/hand.urdf.xacro"/>
@@ -13,11 +13,11 @@
         <mesh filename="package://yanu_description/meshes/yanu.stl" scale="0.001 0.001 0.001"/>
       </geometry>
-	<material name="green"/>
+      <material name="green"/>
     </visual>
-      <collision>
-        <geometry>
-          <mesh filename="package://yanu_description/meshes/yanu.stl" scale="0.001 0.001 0.001"/>
-        </geometry>
-      </collision>
+    <collision>
+      <geometry>
+        <mesh filename="package://yanu_description/meshes/yanu.stl" scale="0.001 0.001 0.001"/>
+      </geometry>
+    </collision>
   </link>
   <joint name="yanu_base_to_panda" type="fixed">
