Commit message: rename from yanu_base_link to base_link

File: urdf/yanu.urdf.xacro (robot description, xacro)
@@ -7,5 +7,5 @@
     <color rgba="0 1 0.0 1"/>
   </material>
-  <link name="yanu_base_link">
+  <link name="base_link">
     <visual>
       <origin rpy="0 0 0" xyz="0 0 0.826"/>
@@ -22,5 +22,5 @@
   </link>
   <joint name="yanu_base_to_panda" type="fixed">
-    <parent link="yanu_base_link"/>
+    <parent link="base_link"/>
     <child link="panda_link0"/>
     <origin xyz="0 0 0.826" rpy="0 0 0"/>
